File: T00R1/Design/T00R10.sch (EAGLE design)
At the start: 1 part, among them P1 HEXABIT_17.32_TRIG_P1_P6

Commit message: -Update the Schematic logo -extended the exposed copper space of the power pads at the angles
Other:
- note added: "T00R1"
- note added: "T00R1_Frontend"
- note removed: "0"
- note removed: "T00R10"
- note removed: "T00R10_Frontend"
